File: ZVS-circut-project.kicad_pcb (KiCad board)
At the start: 2 copper layers, 133.9 x 58 mm, 17 parts, among them J1 691137710002, J2 691137710002, U1 IRFP260NPBF, U2 IRFP260NPBF

Commit message: Add files via upload
Parts:
- moved J2 11.9 mm to (207.4, 85.9), turned to 90 degrees
- moved J1 5.13 mm to (96.7, 82.4), turned to -90 degrees
Connections:
- net Net-(D3-A) renamed /MOSFET RIGHT
- net Net-(D4-A) renamed /MOSFET LEFT
- J1 pad 1: GND -> +12V
- J1 pad 2: +12V -> GND
- J2 pad 1: Net-(D4-K) -> Net-(D3-K)
- J2 pad 2: Net-(D3-K) -> Net-(D4-K)
Routing:
- net Net-(D4-K): track 146.5 -> 135.3 mm
- net Net-(D3-K): track 144.9 -> 134.1 mm
- net +12V: track 204.8 -> 198.9 mm
- net /MOSFET RIGHT: track 35.9 -> 39.2 mm
Other:
- board size 133.9 x 58 mm -> 123.2 x 58 mm
