File: ZVS-circut-project.kicad_sch (KiCad schematic)
At the start: 17 parts, among them J1 691137710002, J2 691137710002, U1 IRFP260NPBF, U2 IRFP260NPBF

Commit message: Add files via upload
Connections:
- net +12V: now also J1.1; no longer J1.2
- net GND: now also J1.2; no longer J1.1
- net MOSFET LEFT: now reaches CR1.1, D4.2 (A), R2.1, R3.2, U2.1 (G)
- net MOSFET RIGHT: now reaches CR2.1, D3.2 (A), R1.2, R5.2, U1.1 (G)
- net at C1.2, D4.1 (K), L1.2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: now also J2.2; no longer J2.1
- net at C1.1, D3.1 (K), L2.1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: now also J2.1; no longer J2.2
Changed lines of the file:
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@@
+    (stroke (width 0) (type default))
+  )
+  (wire (pts (xy 153.67 60.96) (xy 161.29 60.96))
     (stroke (width 0) (type default))
   )
@@
     (stroke (width 0) (type default))
   )
-  (wire (pts (xy 147.32 60.96) (xy 161.29 60.96))
+  (wire (pts (xy 156.21 63.5) (xy 161.29 63.5))
     (stroke (width 0) (type default))
   )
@@
     (stroke (width 0) (type default))
   )
-  (wire (pts (xy 147.32 45.72) (xy 147.32 60.96))
-    (stroke (width 0) (type default))
-  )
-  (wire (pts (xy 147.32 63.5) (xy 161.29 63.5))
-    (stroke (width 0) (type default))
-  )
-  (wire (pts (xy 147.32 63.5) (xy 147.32 80.01))
-    (stroke (width 0) (type default))
-  )
   (wire (pts (xy 123.19 29.21) (xy 123.19 43.18))
     (stroke (width 0) (type default))
@@
     (stroke (width 0) (type default))
   )
-  (wire (pts (xy 134.62 45.72) (xy 147.32 45.72))
-    (stroke (width 0) (type default))
-  )
-  (wire (pts (xy 134.62 80.01) (xy 147.32 80.01))
+  (wire (pts (xy 134.62 45.72) (xy 156.21 45.72))
+    (stroke (width 0) (type default))
+  )
+  (wire (pts (xy 156.21 45.72) (xy 156.21 63.5))
+    (stroke (width 0) (type default))
+  )
+  (wire (pts (xy 134.62 80.01) (xy 153.67 80.01))
     (stroke (width 0) (type default))
   )
@@
     (stroke (width 0) (type default))
   )
+  (wire (pts (xy 153.67 80.01) (xy 153.67 60.96))
+    (stroke (width 0) (type default))
+  )
   (wire (pts (xy 124.46 82.55) (xy 130.81 82.55))
     (stroke (width 0) (type default))
+  )
+  (label "MOSFET LEFT" (at 87.63 74.93 0) (fields_autoplaced)
+    (effects (font (size 1.27 1.27)) (justify left bottom))
+  )
+  (label "MOSFET RIGHT" (at 87.63 49.53 0) (fields_autoplaced)
+    (effects (font (size 1.27 1.27)) (justify left bottom))
   )
   (symbol (lib_id "CF14JT10K0:CF14JT10K0") (at 78.74 74.93 90) (unit 1)
@@
     )
   )
-  (symbol (lib_id "power:+12V") (at 22.86 41.91 90) (unit 1)
-    (in_bom yes) (on_board yes) (dnp no) (fields_autoplaced)
-    (property "Reference" "#PWR05" (at 26.67 41.91 0)
-      (effects (font (size 1.27 1.27)) hide)
-    )
-    (property "Value" "+12V" (at 19.05 41.91 90)
+  (symbol (lib_id "power:+12V") (at 22.86 39.37 90) (unit 1)
+    (in_bom yes) (on_board yes) (dnp no) (fields_autoplaced)
+    (property "Reference" "#PWR05" (at 26.67 39.37 0)
+      (effects (font (size 1.27 1.27)) hide)
+    )
+    (property "Value" "+12V" (at 19.05 39.37 90)
       (effects (font (size 1.27 1.27)) (justify left))
     )
-    (property "Footprint" "" (at 22.86 41.91 0)
-      (effects (font (size 1.27 1.27)) hide)
-    )
-    (property "Datasheet" "" (at 22.86 41.91 0)
+    (property "Footprint" "" (at 22.86 39.37 0)
+      (effects (font (size 1.27 1.27)) hide)
+    )
+    (property "Datasheet" "" (at 22.86 39.37 0)
       (effects (font (size 1.27 1.27)) hide)
     )
@@
     )
   )
-  (symbol (lib_id "power:GND") (at 22.86 39.37 270) (unit 1)
-    (in_bom yes) (on_board yes) (dnp no) (fields_autoplaced)
-    (property "Reference" "#PWR04" (at 16.51 39.37 0)
-      (effects (font (size 1.27 1.27)) hide)
-    )
-    (property "Value" "GND" (at 19.05 39.37 90)
+  (symbol (lib_id "power:GND") (at 22.86 41.91 270) (unit 1)
+    (in_bom yes) (on_board yes) (dnp no) (fields_autoplaced)
+    (property "Reference" "#PWR04" (at 16.51 41.91 0)
+      (effects (font (size 1.27 1.27)) hide)
+    )
+    (property "Value" "GND" (at 19.05 41.91 90)
       (effects (font (size 1.27 1.27)) (justify right))
     )
-    (property "Footprint" "" (at 22.86 39.37 0)
-      (effects (font (size 1.27 1.27)) hide)
-    )
-    (property "Datasheet" "" (at 22.86 39.37 0)
-      (effects (font (size 1.27 1.27)) hide)
-    )
+    (property "Footprint" "" (at 22.86 41.91 0)
+      (effects (font (size 1.27 1.27)) hide)
+    )
+    (property "Datasheet" "" (at 22.86 41.91 0)
+      (effects (font (size 1.27 1.27)) hide)
+    )
